Commit message: Add files via upload

File: diff_bot_description/urdf/diff_bot.xacro (robot description, xacro)
@@ -94,5 +94,5 @@
   <parent link="base_link"/>
   <child link="right_wheel_1"/>
-  <axis xyz="0.0 -1.0 0.0"/>
+  <axis xyz="0.0 1.0 0.0"/>
 </joint>
 <joint name="lidar_joint" type="continuous">
